File: schematics/src/ioboard/YUSynth-LFO-ioboard.sch (EAGLE design)
At the start: 1 part, among them IC1 TL074P

Commit message: initial designs
Parts:
- added ACT_LED: (no value), led:LED5MM
- added C2: 10nF, rcl:C-EU050-024X044
- added CV, PULSE, RAMP, SAW, SINE, SYNC, TRI: WQP-PJ301M-12_JACK, thonkiconn:WQP-PJ301M-12_JACK
- added CV_ATTN: 50k lin, TomW:ALPHA-9MMA
- added INPUT_CON: (no value), pinhead:PINHD-1X2
- added LOWEST_RATE: 50k, rcl:R-TRIMM64X
- added OUTPUT_CON: (no value), pinhead:PINHD-1X6
- added PULSE_WIDTH, RATE: 10k lin, TomW:ALPHA-9MMA
- added PWR_CON: (no value), pinhead:PINHD-1X3
- added Q1: BS170, transistor-small-signal:BS170
- added R1, R3: 15k, rcl:R-US_0207/7
- added R10, R11, R12, R5, R9: 100k, rcl:R-US_0207/7
- added R14: 12k, rcl:R-US_0207/7
- added R16: 1k, rcl:R-US_0207/7
- added R4: 10k, rcl:R-US_0207/7
- added R6: 8.2k, rcl:R-US_0207/7
- added R7: 27k, rcl:R-US_0207/7
- added R8: 820R, rcl:R-US_0207/7
- added T1: (no value), transistor:BC557C-PNP-TO92-EBC
- added T2: (no value), transistor:BC547-NPN-TO92-CBE
- IC1: value TL074P -> LM741P; device linear:TL074P -> linear:LM741P
Connections:
- new net +12V: IC1.V+, LOWEST_RATE.E, PWR_CON.1, R1.2, R14.1, R8.1, T1.E, T2.C
- new net -12V: IC1.V-, PWR_CON.3, R3.1
- new net CV: INPUT_CON.1, Q1.D, T1.C
- new net GND: ACT_LED.C, CV.1, CV_ATTN.A, LOWEST_RATE.A, PULSE.1, PWR_CON.2, Q1.S, R5.2, R6.2, RAMP.1, RATE.A, SAW.1, SINE.1, SYNC.1, TRI.1
- new net LED: OUTPUT_CON.6, T2.B
- new net N$1: PULSE_WIDTH.A, R3.2
- new net N$10: R14.2, RATE.E
- new net N$11: R10.2, RATE.S
- new net N$13: IC1.-IN, R10.1, R11.1, R12.1, R9.2
- new net N$14: LOWEST_RATE.S, R11.2
- new net N$15: CV_ATTN.S, R12.2
- new net N$16: CV.2, CV_ATTN.E
- new net N$17: R16.1, T2.E
- new net N$18: ACT_LED.A, R16.2
- new net N$2: PULSE_WIDTH.E, R1.1
- new net N$3: C2.1, SYNC.2
- new net N$4: C2.2, R4.2
- new net N$5: Q1.G, R4.1, R5.1
- new net N$7: IC1.+IN, R6.1
- new net N$8: IC1.OUT, R7.2, R9.1
- new net N$9: R7.1, R8.2, T1.B
- new net PULSE_OUT: OUTPUT_CON.4, PULSE.2
- new net PULSE_WIDTH: INPUT_CON.2, PULSE_WIDTH.S
- new net RAMP_OUT: OUTPUT_CON.1, RAMP.2
- new net SAW_OUT: OUTPUT_CON.5, SAW.2
- new net SINE_OUT: OUTPUT_CON.3, SINE.2
- new net TRI_OUT: OUTPUT_CON.2, TRI.2
