File: schematics/src/ioboard/ioboard.brd (EAGLE design)
At the start: 48.3 x 99.1 mm, 33 parts, among them IC1 LM741P, Q1 BS170

Commit message: Added files & structure
Parts:
- moved SAW 19.1 mm to (7.62, 7.62), turned to 180 degrees
- moved TRI 19.1 mm to (7.62, 26.7), turned to 0 degrees
- moved R11 6.98 mm to (17.1, 87.6)
- moved LOWEST_RATE 3.81 mm to (6.35, 95.2)
Routing:
- net SAW_OUT: track 57.5 -> 89.2 mm
- net TRI_OUT: track 90.5 -> 63.7 mm
- net N$14: track 5.08 -> 13.6 mm
- net N$13: track 72.6 -> 65.6 mm
- net +12V: track 139.6 -> 141.2 mm
Changed lines of the file:
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@@
 <attribute name="VALUE" x="21.844" y="83.2612" size="1.27" layer="27" ratio="10"/>
 </element>
-<element name="R11" library="rcl" library_urn="urn:adsk.eagle:library:334" package="0207/7" package3d_urn="urn:adsk.eagle:package:23493/2" value="100k" x="10.16" y="87.63" smashed="yes" rot="R90">
-<attribute name="NAME" x="10.795" y="85.09" size="1.27" layer="25" font="vector" ratio="10" rot="R90"/>
-<attribute name="POPULARITY" value="22" x="10.16" y="87.63" size="1.778" layer="27" rot="R90" display="off"/>
-<attribute name="SPICEPREFIX" value="R" x="10.16" y="87.63" size="1.778" layer="27" rot="R90" display="off"/>
-<attribute name="VALUE" x="10.7188" y="85.344" size="1.27" layer="27" ratio="10" rot="R90"/>
+<element name="R11" library="rcl" library_urn="urn:adsk.eagle:library:334" package="0207/7" package3d_urn="urn:adsk.eagle:package:23493/2" value="100k" x="17.145" y="87.63" smashed="yes" rot="R90">
+<attribute name="NAME" x="17.78" y="85.09" size="1.27" layer="25" font="vector" ratio="10" rot="R90"/>
+<attribute name="POPULARITY" value="22" x="17.145" y="87.63" size="1.778" layer="27" rot="R90" display="off"/>
+<attribute name="SPICEPREFIX" value="R" x="17.145" y="87.63" size="1.778" layer="27" rot="R90" display="off"/>
+<attribute name="VALUE" x="17.7038" y="85.344" size="1.27" layer="27" ratio="10" rot="R90"/>
 </element>
 <element name="R12" library="rcl" library_urn="urn:adsk.eagle:library:334" package="0207/7" package3d_urn="urn:adsk.eagle:package:23493/2" value="100k" x="21.59" y="54.61" smashed="yes" rot="R180">
@@
 </element>
 <element name="RATE" library="TomW" package="EVUF" value="10k lin" x="24.13" y="96.52" smashed="yes">
-<attribute name="NAME" x="29.21" y="88.9" size="1.778" layer="25" font="vector" ratio="10"/>
+<attribute name="NAME" x="31.115" y="96.52" size="1.778" layer="25" font="vector" ratio="10"/>
 <attribute name="VALUE" x="20.32" y="92.71" size="1.27" layer="27"/>
 </element>
@@
 <attribute name="VALUE" x="21.844" y="85.8012" size="1.27" layer="27" ratio="10"/>
 </element>
-<element name="LOWEST_RATE" library="rcl" library_urn="urn:adsk.eagle:library:334" package="RTRIM64X" package3d_urn="urn:adsk.eagle:package:23749/1" value="50k" x="10.16" y="95.25" smashed="yes" rot="R90">
-<attribute name="NAME" x="15.875" y="97.79" size="1.27" layer="25" font="vector" ratio="10" rot="R270"/>
-<attribute name="POPULARITY" value="2" x="10.16" y="95.25" size="1.778" layer="27" rot="R90" display="off"/>
-<attribute name="SPICEMODEL" value="X" x="10.16" y="95.25" size="1.778" layer="27" rot="R90" display="off"/>
-<attribute name="SPICEPREFIXL" value="POT" x="10.16" y="95.25" size="1.778" layer="27" rot="R90" display="off"/>
-<attribute name="VALUE" x="13.56" y="95.32" size="1.27" layer="27" rot="R180"/>
+<element name="LOWEST_RATE" library="rcl" library_urn="urn:adsk.eagle:library:334" package="RTRIM64X" package3d_urn="urn:adsk.eagle:package:23749/1" value="50k" x="6.35" y="95.25" smashed="yes" rot="R90">
+<attribute name="NAME" x="1.27" y="91.44" size="1.27" layer="25" font="vector" ratio="10"/>
+<attribute name="POPULARITY" value="2" x="6.35" y="95.25" size="1.778" layer="27" rot="R90" display="off"/>
+<attribute name="SPICEMODEL" value="X" x="6.35" y="95.25" size="1.778" layer="27" rot="R90" display="off"/>
+<attribute name="SPICEPREFIXL" value="POT" x="6.35" y="95.25" size="1.778" layer="27" rot="R90" display="off"/>
+<attribute name="VALUE" x="9.75" y="95.32" size="1.27" layer="27" rot="R180"/>
 </element>
 <element name="CV" library="thonkiconn" package="WQP-PJ301M-12_JACK" value="" x="7.62" y="66.04" smashed="yes" rot="R180">
@@
 <attribute name="NAME" x="35.56" y="8.255" size="1.27" layer="25" font="vector" ratio="10" rot="R90"/>
 </element>
-<element name="TRI" library="thonkiconn" package="WQP-PJ301M-12_JACK" value="" x="7.62" y="7.62" smashed="yes" rot="R180">
-<attribute name="NAME" x="2.54" y="9.525" size="1.27" layer="25" font="vector" ratio="10" rot="R90"/>
+<element name="TRI" library="thonkiconn" package="WQP-PJ301M-12_JACK" value="" x="7.62" y="26.67" smashed="yes">
+<attribute name="NAME" x="2.54" y="29.845" size="1.27" layer="25" font="vector" ratio="10" rot="R90"/>
 </element>
 <element name="PULSE" library="thonkiconn" package="WQP-PJ301M-12_JACK" value="" x="24.13" y="26.67" smashed="yes">
 <attribute name="NAME" x="19.05" y="27.94" size="1.27" layer="25" font="vector" ratio="10" rot="R90"/>
 </element>
-<element name="SAW" library="thonkiconn" package="WQP-PJ301M-12_JACK" value="" x="7.62" y="26.67" smashed="yes">
-<attribute name="NAME" x="2.54" y="29.21" size="1.27" layer="25" font="vector" ratio="10" rot="R90"/>
+<element name="SAW" library="thonkiconn" package="WQP-PJ301M-12_JACK" value="" x="7.62" y="7.62" smashed="yes" rot="R180">
+<attribute name="NAME" x="2.54" y="8.255" size="1.27" layer="25" font="vector" ratio="10" rot="R90"/>
 </element>
 <element name="PWR_CON" library="pinhead" library_urn="urn:adsk.eagle:library:325" package="1X03" package3d_urn="urn:adsk.eagle:package:22458/2" value="" x="33.02" y="16.51" smashed="yes" rot="R270">
@@
 <contactref element="T2" pad="C"/>
 <contactref element="PWR_CON" pad="1"/>
-<wire x1="7.62" y1="96.52" x2="7.62" y2="91.44" width="0.6096" layer="16"/>
-<wire x1="7.62" y1="91.44" x2="10.16" y2="88.9" width="0.6096" layer="16"/>
+<wire x1="3.81" y1="96.52" x2="3.81" y2="95.25" width="0.6096" layer="16"/>
+<wire x1="3.81" y1="95.25" x2="10.16" y2="88.9" width="0.6096" layer="16"/>
 <wire x1="10.16" y1="88.9" x2="17.78" y2="88.9" width="0.6096" layer="16"/>
 <wire x1="17.78" y1="88.9" x2="20.32" y2="86.36" width="0.6096" layer="16"/>
@@
 <contactref element="R10" pad="1"/>
 <contactref element="R11" pad="1"/>
-<wire x1="10.16" y1="83.82" x2="20.32" y2="83.82" width="0.4064" layer="1"/>
+<wire x1="17.145" y1="83.82" x2="20.32" y2="83.82" width="0.4064" layer="1"/>
 <wire x1="10.16" y1="49.53" x2="8.89" y2="49.53" width="0.4064" layer="16"/>
 <wire x1="8.89" y1="49.53" x2="7.62" y2="48.26" width="0.4064" layer="16"/>
@@
 <contactref element="LOWEST_RATE" pad="2"/>
 <contactref element="R11" pad="2"/>
-<wire x1="10.16" y1="91.44" x2="10.16" y2="96.52" width="0.4064" layer="1"/>
+<wire x1="17.145" y1="91.44" x2="10.16" y2="91.44" width="0.4064" layer="1"/>
+<wire x1="10.16" y1="91.44" x2="6.35" y2="95.25" width="0.4064" layer="1"/>
+<wire x1="6.35" y1="95.25" x2="6.35" y2="96.52" width="0.4064" layer="1"/>
 </signal>
 <signal name="N$15">
@@
 <contactref element="TRI" pad="P$1"/>
 <contactref element="OUTPUT_CON" pad="2"/>
-<wire x1="7.62" y1="2.62" x2="7.62" y2="8.89" width="0.4064" layer="16"/>
-<wire x1="7.62" y1="8.89" x2="12.7" y2="13.97" width="0.4064" layer="16"/>
+<wire x1="7.62" y1="31.67" x2="7.62" y2="31.75" width="0.4064" layer="16"/>
+<wire x1="7.62" y1="31.75" x2="8.89" y2="33.02" width="0.4064" layer="16"/>
 <wire x1="12.7" y1="33.02" x2="15.24" y2="35.56" width="0.4064" layer="16"/>
 <wire x1="15.24" y1="35.56" x2="15.24" y2="43.18" width="0.4064" layer="16"/>
-<wire x1="12.7" y1="13.97" x2="12.7" y2="33.02" width="0.4064" layer="16"/>
+<wire x1="8.89" y1="33.02" x2="12.7" y2="33.02" width="0.4064" layer="16"/>
 <wire x1="15.24" y1="43.18" x2="12.7" y2="45.72" width="0.4064" layer="16"/>
 <wire x1="12.7" y1="45.72" x2="12.7" y2="78.74" width="0.4064" layer="16"/>
@@
 <contactref element="SAW" pad="P$1"/>
 <contactref element="OUTPUT_CON" pad="5"/>
-<wire x1="7.62" y1="31.67" x2="7.62" y2="33.02" width="0.4064" layer="16"/>
-<wire x1="7.62" y1="33.02" x2="5.08" y2="35.56" width="0.4064" layer="16"/>
+<wire x1="7.62" y1="2.62" x2="7.62" y2="6.985" width="0.4064" layer="16"/>
+<wire x1="7.62" y1="6.985" x2="10.795" y2="10.16" width="0.4064" layer="16"/>
+<wire x1="10.795" y1="10.16" x2="10.795" y2="24.13" width="0.4064" layer="16"/>
+<wire x1="10.795" y1="24.13" x2="5.08" y2="29.845" width="0.4064" layer="16"/>
+<wire x1="5.08" y1="85.09" x2="5.08" y2="29.845" width="0.4064" layer="16"/>
 <wire x1="5.08" y1="85.09" x2="3.81" y2="86.36" width="0.4064" layer="16"/>
 <wire x1="3.81" y1="86.36" x2="2.54" y2="86.36" width="0.4064" layer="16"/>
-<wire x1="5.08" y1="35.56" x2="5.08" y2="85.09" width="0.4064" layer="16"/>
 </signal>
 <signal name="RAMP_OUT">
