File: schematics/src/mainboard/YUSynth-LFO-mainboard.sch (EAGLE design)
At the start: 42 parts, among them IC1 TL074P, IC2 TL074P, IC3 NE555N

Commit message: initial designs
Parts:
- added C2: 1uF, rcl:C-EU075-032X103
- added INPUT_CON: (no value), pinhead:PINHD-1X2
- added OUTPUT_CON: (no value), pinhead:PINHD-1X6
- added PWR_CON: (no value), pinhead:PINHD-1X3
- added R24, R26: 100k, rcl:R-US_0207/7
- added R25: 47k, rcl:R-US_0207/7
- added R27: 1k, rcl:R-US_0207/7
- added R28: 2.7k, rcl:R-US_0207/7
- added SAW_BIAS: 10k, rcl:R-TRIMM64W
- added SINE/TRI_SYMETRY: 50k, rcl:R-TRIMM64W
- C1: value (none) -> 10nF
- C10, C11, C12, C3, C9: value (none) -> .1uF
- C4: value (none) -> 47nF
- C5: value (none) -> 120pF
- C8: value (none) -> 1nF
- D1, D2, D3, D4: value 4148 -> 1n4148
- R1, R19, R23, R5, R8: value (none) -> 1k
- R10, R6: value (none) -> 10k
- R11, R12, R14, R2: value (none) -> 100k/1%
- R13: value (none) -> 50k/1%
- R15, R3: value (none) -> 200k/1%
- R16, R18: value (none) -> 150k
- R17: value (none) -> 100k; device rcl:R-TRIMM64W -> rcl:R-US_0207/7
- R20: value (none) -> 22k
- R21: value (none) -> 15k
- R22: value (none) -> 1.5k
- R4: value (none) -> 12k
- R7: value (none) -> 120k
- R9: value (none) -> 100k
Connections:
- removed net CV_INPUT: IC1B.+IN, IC3.DIS, IC3.THR, R1.1
- new net CV: C2.1, IC1B.+IN, IC3.DIS, IC3.THR, INPUT_CON.1, R1.1
- new net LED: OUTPUT_CON.6, R25.2
- new net N$21: IC1D.OUT, R11.1, R14.1, R26.1, R8.1, R9.2
- new net N$23: IC2A.OUT, R17.2, R27.1
- new net N$5: IC2A.-IN, R17.1, R26.2
- new net RAMP_OUT: OUTPUT_CON.1, R27.2
- net +12V: now also PWR_CON.1, SINE/TRI_SYMETRY.E; no longer R17.E
- net -12V: now also PWR_CON.3, R28.2
- net GND: now also C2.2, PWR_CON.2, SAW_BIAS.E, SINE/TRI_SYMETRY.A; no longer R17.A
- net LED_OUT: now also R25.1
- net N$10: now also R28.1, SAW_BIAS.A; no longer IC2A.-IN, IC2A.OUT
- net N$16: now also SINE/TRI_SYMETRY.S; no longer R17.S
- net N$4: now also R24.2
- net N$7: now also R24.1, SAW_BIAS.S; no longer IC1D.OUT, R8.1, R9.2
- net N$8: no longer R11.1, R14.1
- net PULSE_OUT: now also OUTPUT_CON.4
- net PULSE_WIDTH: now also INPUT_CON.2
- net SAW_OUT: now also OUTPUT_CON.5
- net SINE_OUT: now also OUTPUT_CON.3
- net TRI_OUT: now also OUTPUT_CON.2
Other:
- moved on the sheet: C1, C10, C11, C12, C3, C4, C5, C6, C7, C8, C9, D1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
