File: schematics/src/mainboard/mainboard.brd (EAGLE design)
At the start: 48.3 x 99.1 mm, 53 parts, among them IC1 TL074P, IC2 TL074P, IC3 NE555N

Commit message: Updated Schematics, Fixed Power Socket orientation
Parts:
- removed C6, C7: 10uf, resistor:E2,5-5
- added C13, C19: 10uf, resistor:E2,5-5
- SAW_BIAS, SINE/TRI_SYMETRY: device rcl:RTRIM64W -> pot:S64YW
- moved SINE/TRI_SYMETRY 8.82 mm to (11.4, 81.9)
- moved C1 3.81 mm to (15.2, 88.9)
- turned PWR to 0 degrees
- turned SAW_BIAS to 180 degrees
Connections:
- net +12V: now also C19.+, PWR.10, PWR.9, SINE/TRI_SYMETRY.E; no longer C7.+, PWR.1, PWR.2, SINE/TRI_SYMETRY.3
- net -12V: now also C13.-, PWR.1, PWR.2; no longer C6.-, PWR.10, PWR.9
- net GND: now also C13.+, C19.-, SAW_BIAS.E, SINE/TRI_SYMETRY.A; no longer C6.+, C7.-, SAW_BIAS.3, SINE/TRI_SYMETRY.1
- net N$10: now also SAW_BIAS.A; no longer SAW_BIAS.1
- net N$16: now also SINE/TRI_SYMETRY.S; no longer SINE/TRI_SYMETRY.2
- net N$7: now also SAW_BIAS.S; no longer SAW_BIAS.2
Routing:
- net N$16: track 2.54 -> 8.04 mm
- net +12V: track 136.5 -> 139.7 mm
- net N$1: track 2.54 -> 4.86 mm
- net -12V: track 84.7 -> 86.6 mm
