File: schematics/src/mainboard/mainboard.sch (EAGLE design)
At the start: 53 parts, among them IC1 TL074P, IC2 TL074P, IC3 NE555N

Commit message: Updated Schematics, Fixed Power Socket orientation
Parts:
- removed C6, C7: 10uf, resistor:CPOL-USE2.5-5
- added C13, C19: 10uf, resistor:CPOL-USE2.5-5
- SAW_BIAS, SINE/TRI_SYMETRY: device rcl:R-TRIMM64W -> pot:TRIM_1234-S64YW
Connections:
- net +12V: now also C19.+, PWR.10, PWR.9; no longer C7.+, PWR.1, PWR.2
- net -12V: now also C13.-, PWR.1, PWR.2; no longer C6.-, PWR.10, PWR.9
- net GND: now also C13.+, C19.-; no longer C6.+, C7.-
Other:
- moved on the sheet: PWR
